Commit message: feat: Implement Arduino Hardware Interface for ROS2
- Updated package.xml to reflect new versioning and dependencies.
- Added arduino_hardware_interface.cpp and arduino_hardware_interface.hpp for core functionality.
- Introduced arduino_hardware_interface.py for Python-based interface.
- Created plugin XML for hardware interface registration.
- Developed scripts for testing Arduino robot with teleoperation.
- Implemented serial communication and encoder reading logic.
- Enhanced command and state interface management for wheel control.

File: description/ros2_control.xacro (robot description, xacro)
@@ -8,5 +8,5 @@
                 <plugin>gazebo_ros2_control/GazeboSystem</plugin>
             </hardware>
-            <joint name="left_wheel_joint">
+            <joint name="base_left_wheel_joint">
                 <command_interface name="velocity">
                     <param name="min">-10</param>
@@ -16,5 +16,5 @@
                 <state_interface name="velocity" />
             </joint>
-            <joint name="right_wheel_joint">
+            <joint name="base_right_wheel_joint">
                 <command_interface name="velocity">
                     <param name="min">-10</param>
@@ -39,14 +39,13 @@
         <ros2_control name="RealRobot" type="system">
             <hardware>
-                <plugin>diffdrive_arduino/DiffDriveArduino</plugin>
-                <param name="left_wheel_name">left_wheel_joint</param>
-                <param name="right_wheel_name">right_wheel_joint</param>
-                <param name="loop_rate">30</param>
-                <param name="device">/dev/ttyUSB0</param>
+                <plugin>arduino_hardware_interface/ArduinoHardwareInterface</plugin>
+                <param name="device">/dev/ttyACM0</param>
                 <param name="baud_rate">57600</param>
                 <param name="timeout">1000</param>
                 <param name="enc_counts_per_rev">3436</param>
+                <param name="wheel_radius">0.065</param>
+                <param name="wheel_separation">0.17</param>
             </hardware>
-            <joint name="left_wheel_joint">
+            <joint name="base_left_wheel_joint">
                 <command_interface name="velocity">
                     <param name="min">-10</param>
@@ -56,5 +55,5 @@
                 <state_interface name="position"/>
             </joint>
-            <joint name="right_wheel_joint">
+            <joint name="base_right_wheel_joint">
                 <command_interface name="velocity">
                     <param name="min">-10</param>
