Commit message: Add launch files and configuration for ROS2 control and simulation support

File: description/robot.urdf.xacro (robot description, xacro)
@@ -1,9 +1,16 @@
 <?xml version="1.0"?>
 <robot xmlns:xacro="http://www.ros.org/wiki/xacro"  name="robot">
+    <!-- Argomenti per configurazione -->
+    <xacro:arg name="use_ros2_control" default="true" />
+    <xacro:arg name="sim_mode" default="false" />
     <xacro:include filename="robot_core.xacro" />
-    <!-- simulation with gazebo controller (for odom)-->
-    <xacro:include filename="gazebo_control.xacro" />
-    <!-- real robot (for odom)-->
-    <!-- <xacro:include filename="ros2_control.xacro" /> -->
+    <!-- ROS2 Control (sia per simulazione che reale) -->
+    <xacro:if value="$(arg use_ros2_control)">
+        <xacro:include filename="ros2_control.xacro" />
+    </xacro:if>
+    <!-- Gazebo control legacy (solo se non si usa ros2_control) -->
+    <xacro:unless value="$(arg use_ros2_control)">
+        <xacro:include filename="gazebo_control.xacro" />
+    </xacro:unless>
     <xacro:include filename="lidar.xacro" />
     <xacro:include filename="camera.xacro" />

File: description/ros2_control.xacro (robot description, xacro)
@@ -1,64 +1,68 @@
 <?xml version="1.0"?>
 <robot xmlns:xacro="http://www.ros.org/wiki/xacro" >
-    <!-- GAZEBO CONTROL MANAGER-->
-    <!-- <ros2_control name="GazeboSystem" type="system">
-    <hardware>
-        <plugin>gazebo_ros2_control/GazeboSystem</plugin>
-    </hardware>
-    <joint name="left_wheel_joint">
-        <command_interface name="velocity">
-            <param name="min">-10</param>
-            <param name="max">10</param>
-        </command_interface>
-        <state_interface name="position" />
-        <state_interface name="velocity" />
-    </joint>
-    <joint name="right_wheel_joint">
-        <command_interface name="velocity">
-            <param name="min">-10</param>
-            <param name="max">10</param>
-        </command_interface>
-        <state_interface name="velocity" />
-        <state_interface name="position" />
-    </joint>
-  </ros2_control>  -->
-  <!-- Controllers-->
-  <!-- Ruote-->
-  <gazebo>
-    <plugin filename="libgazebo_ros2_control.so" name="gazebo_ros2_control">
-        <parameters>$(find robot_ros)/description/config/my_controllers.yaml</parameters>
-    </plugin>
-  </gazebo>
-  <!-- REAL CONTROL MANAGER-->
-  <!-- In https://articulatedrobotics.xyz/mobile-robot-13-ros2-control-real/ the DiffDriveArduino has been used-->
-  <!-- but it has to be installed and used with an Arduino Nano as hardware interface -->
-  <!--  -->
-  <!-- <ros2_control name="RealRobot" type="system">
-    <hardware>
-        <plugin>diffdrive_arduino/DiffDriveArduino</plugin>
-        <param name="left_wheel_name">left_wheel_joint</param>
-        <param name="right_wheel_name">right_wheel_joint</param>
-        <param name="loop_rate">30</param>
-        <param name="device">/dev/ttyUSB0</param>
-        <param name="baud_rate">57600</param>
-        <param name="timeout">1000</param>
-        <param name="enc_counts_per_rev">3436</param>
-    </hardware>
-    <joint name="left_wheel_joint">
-        <command_interface name="velocity">
-            <param name="min">-10</param>
-            <param name="max">10</param>
-        </command_interface>
-        <state_interface name="velocity"/>
-        <state_interface name="position"/>
-    </joint>
-    <joint name="right_wheel_joint">
-        <command_interface name="velocity">
-            <param name="min">-10</param>
-            <param name="max">10</param>
-        </command_interface>
-        <state_interface name="velocity"/>
-        <state_interface name="position"/>
-    </joint>
-  </ros2_control> -->
+    <xacro:arg name="sim_mode" default="false" />
+    <!-- GAZEBO CONTROL MANAGER (per simulazione) -->
+    <xacro:if value="$(arg sim_mode)">
+        <ros2_control name="GazeboSystem" type="system">
+            <hardware>
+                <plugin>gazebo_ros2_control/GazeboSystem</plugin>
+            </hardware>
+            <joint name="left_wheel_joint">
+                <command_interface name="velocity">
+                    <param name="min">-10</param>
+                    <param name="max">10</param>
+                </command_interface>
+                <state_interface name="position" />
+                <state_interface name="velocity" />
+            </joint>
+            <joint name="right_wheel_joint">
+                <command_interface name="velocity">
+                    <param name="min">-10</param>
+                    <param name="max">10</param>
+                </command_interface>
+                <state_interface name="velocity" />
+                <state_interface name="position" />
+            </joint>
+        </ros2_control>
+    </xacro:if>
+    <!-- Controllers per Gazebo -->
+    <xacro:if value="$(arg sim_mode)">
+        <gazebo>
+            <plugin filename="libgazebo_ros2_control.so" name="gazebo_ros2_control">
+                <parameters>$(find robot_ros)/config/my_controllers.yaml</parameters>
+                <parameters>$(find robot_ros)/config/gaz_ros2_ctl_sim.yaml</parameters>
+            </plugin>
+        </gazebo>
+    </xacro:if>
+    <!-- REAL CONTROL MANAGER (per robot reale) -->
+    <xacro:unless value="$(arg sim_mode)">
+        <ros2_control name="RealRobot" type="system">
+            <hardware>
+                <plugin>diffdrive_arduino/DiffDriveArduino</plugin>
+                <param name="left_wheel_name">left_wheel_joint</param>
+                <param name="right_wheel_name">right_wheel_joint</param>
+                <param name="loop_rate">30</param>
+                <param name="device">/dev/ttyUSB0</param>
+                <param name="baud_rate">57600</param>
+                <param name="timeout">1000</param>
+                <param name="enc_counts_per_rev">3436</param>
+            </hardware>
+            <joint name="left_wheel_joint">
+                <command_interface name="velocity">
+                    <param name="min">-10</param>
+                    <param name="max">10</param>
+                </command_interface>
+                <state_interface name="velocity"/>
+                <state_interface name="position"/>
+            </joint>
+            <joint name="right_wheel_joint">
+                <command_interface name="velocity">
+                    <param name="min">-10</param>
+                    <param name="max">10</param>
+                </command_interface>
+                <state_interface name="velocity"/>
+                <state_interface name="position"/>
+            </joint>
+        </ros2_control>
+    </xacro:unless>
 </robot>

Commit message: feat: Implement complete integration of ros2_control with Arduino Nano and L298N
- Added new Arduino sketch for hardware interface with encoder support and motor control.
- Configured ros2_control with DiffDriveArduino plugin and updated URDF for real robot integration.
- Enhanced launch files to include controller manager and joint state broadcaster for improved control flow.
- Created comprehensive documentation including wiring guide, deployment guide, and Arduino README.
- Deprecated custom hardware interface nodes in favor of ros2_control.
- Made LIDAR serial port configurable via launch arguments for flexibility.
- Established a clear architecture for the robot system, detailing data flow and TF frames.

File: description/robot.urdf.xacro (robot description, xacro)
@@ -3,7 +3,7 @@
     <xacro:include filename="robot_core.xacro" />
     <!-- simulation with gazebo controller (for odom)-->
-    <xacro:include filename="gazebo_control.xacro" />
+    <!-- <xacro:include filename="gazebo_control.xacro" /> -->
     <!-- real robot (for odom)-->
-    <!-- <xacro:include filename="ros2_control.xacro" /> -->
+    <xacro:include filename="ros2_control.xacro" />
     <xacro:include filename="lidar.xacro" />
     <xacro:include filename="camera.xacro" />

File: description/ros2_control.xacro (robot description, xacro)
@@ -1,38 +1,7 @@
 <?xml version="1.0"?>
 <robot xmlns:xacro="http://www.ros.org/wiki/xacro" >
-    <!-- GAZEBO CONTROL MANAGER-->
-    <!-- <ros2_control name="GazeboSystem" type="system">
-    <hardware>
-        <plugin>gazebo_ros2_control/GazeboSystem</plugin>
-    </hardware>
-    <joint name="left_wheel_joint">
-        <command_interface name="velocity">
-            <param name="min">-10</param>
-            <param name="max">10</param>
-        </command_interface>
-        <state_interface name="position" />
-        <state_interface name="velocity" />
-    </joint>
-    <joint name="right_wheel_joint">
-        <command_interface name="velocity">
-            <param name="min">-10</param>
-            <param name="max">10</param>
-        </command_interface>
-        <state_interface name="velocity" />
-        <state_interface name="position" />
-    </joint>
-  </ros2_control>  -->
-  <!-- Controllers-->
-  <!-- Ruote-->
-  <gazebo>
-    <plugin filename="libgazebo_ros2_control.so" name="gazebo_ros2_control">
-        <parameters>$(find robot_ros)/description/config/my_controllers.yaml</parameters>
-    </plugin>
-  </gazebo>
-  <!-- REAL CONTROL MANAGER-->
-  <!-- In https://articulatedrobotics.xyz/mobile-robot-13-ros2-control-real/ the DiffDriveArduino has been used-->
-  <!-- but it has to be installed and used with an Arduino Nano as hardware interface -->
-  <!--  -->
-  <!-- <ros2_control name="RealRobot" type="system">
+  <!-- REAL ROBOT CONTROL MANAGER con Arduino Nano -->
+  <!-- Hardware interface per robot reale con encoder -->
+  <ros2_control name="RealRobot" type="system">
     <hardware>
         <plugin>diffdrive_arduino/DiffDriveArduino</plugin>
@@ -43,5 +12,5 @@
         <param name="baud_rate">57600</param>
         <param name="timeout">1000</param>
-        <param name="enc_counts_per_rev">3436</param>
+        <param name="enc_counts_per_rev">374</param>
     </hardware>
     <joint name="left_wheel_joint">
@@ -61,4 +30,4 @@
         <state_interface name="position"/>
     </joint>
-  </ros2_control> -->
+  </ros2_control>
 </robot>
